Commit message: misc updates

File: urdf/blocky.urdf.xacro (robot description, xacro)
@@ -3,4 +3,5 @@
   <!-- Set up some variables and defaults -->
   <xacro:property name="width" value="0.2" />
+  <xacro:property name="pi" value="3.1415" />
   <material name="blue">
     <color rgba="0 0 0.8 1"/>
@@ -16,5 +17,6 @@
   </xacro:macro>
   <!-- Define Links-->
-  <link name="base_link">
+  <link name="base_link" />
+  <link name="link1">
     <visual>
       <geometry>
@@ -30,5 +32,5 @@
     <xacro:default_inertial mass="10"/>
   </link>
-  <link name="head">
+  <link name="link2">
     <visual>
       <geometry>
@@ -45,10 +47,16 @@
   </link>
   <!-- Define Joints -->
+  <joint name="joint0" type="fixed">
+    <parent link="base_link"/>
+    <child link="link1"/>
+    <axis xyz="0 0 1"/>
+    <origin xyz="0 0 0"/>
+  </joint>
   <joint name="joint1" type="continuous">
-    <parent link="base_link"/>
-    <child link="head"/>
+    <parent link="link1"/>
+    <child link="link2"/>
     <axis xyz="0 0 1"/>
     <origin xyz="0 0 ${width}"/>
-    <limit effort="30" velocity="1.0"/>
+    <limit effort="30" velocity="10" lower="0" upper="${pi*2}"/>
   </joint>
   <!-- Define Transmissions -->
@@ -59,5 +67,5 @@
     </actuator>
     <joint name="joint1">
-      <hardwareInterface>PositionJointInterface</hardwareInterface>
+      <hardwareInterface>hardware_interface/PositionJointInterface</hardwareInterface>
     </joint>
   </transmission>
